File: Hardware/Controller/ClockClock24.kicad_pcb (KiCad board)
At the start: 4 copper layers, 78.9 x 51 mm, 45 parts, among them J1 USB_C_Receptacle_USB2.0_16P, J2 BUS_IN, J3 BUS_OUT, J4 CLK1, J5 CLK3, J6 CLK2, J7 CLK4, SW1 SW_Push, SW2 SW_Push, U1 USBLC6-2SC6, U2 ESP32-S3-WROOM-1, U3 AP7361C-33E, U4 VID6606, U5 VID6606

Commit message: added images
Other:
- board text added: "ClockClock24 v 1.0"

Commit message: Add Motor_PCB board and update Controller
- New Motor_PCB KiCad project (motor-only board), linked to Kicad_Libs
- Controller: schematic, PCB and project updates
Parts:
- added C12: 1u, eCapacitor:0603, F.Cu at (91.3, 102.5)
Connections:
- J6 pad 1: /C1 -> /C3
- J6 pad 2: /C2 -> /C4
- J6 pad 3: /C4 -> /C2
- J6 pad 4: /C3 -> /C1
- J6 pad 5: /D1 -> /D3
- J6 pad 6: /D2 -> /D4
- J6 pad 7: /D4 -> /D2
- J6 pad 8: /D3 -> /D1
- J7 pad 1: /G1 -> /G3
- J7 pad 2: /G2 -> /G4
- J7 pad 3: /G4 -> /G2
- J7 pad 4: /G3 -> /G1
- J7 pad 5: /H1 -> /H3
- J7 pad 6: /H2 -> /H4
- J7 pad 7: /H4 -> /H2
- J7 pad 8: /H3 -> /H1
Routing:
- net /C1: track 25.3 -> 37.0 mm
- net /H1: track 18.3 -> 29.3 mm
- net /G1: track 23.3 -> 33.6 mm
- net /D2: track 10.0 -> 19.0 mm
- net /H2: track 18.5 -> 25.3 mm
- net /H3: track 19.8 -> 14.2 mm, vias 0 -> 1
- net /D1: track 9.74 -> 15.1 mm, vias 0 -> 1
- net /D3: track 10.6 -> 15.0 mm
- net /C2: track 25.0 -> 21.1 mm
- net /C4: track 24.7 -> 21.9 mm
- net /G4: track 24.0 -> 21.3 mm, vias 1 -> 2
- net /C3: track 24.4 -> 26.9 mm
- net /H4: track 19.3 -> 17.0 mm
- net /G2: track 23.6 -> 25.4 mm, vias 1 -> 2
- net Net-(U2-IO0): track 6.65 -> 8.30 mm
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
Commit message: Added Fab files, BOM and minor changes in layout
Routing:
- net /USB_D+: track 7.19 -> 7.93 mm
