File: Hardware/Controller/ClockClock24.kicad_sch (KiCad schematic)
At the start: 45 parts, among them J1 USB_C_Receptacle_USB2.0_16P, J2 BUS_IN, J3 BUS_OUT, J4 CLK1, J5 CLK3, J6 CLK2, J7 CLK4, SW1 SW_Push, SW2 SW_Push, U1 USBLC6-2SC6, U2 ESP32-S3-WROOM-1, U3 AP7361C-33E, U4 VID6606, U5 VID6606

Commit message: Add Motor_PCB board and update Controller
- New Motor_PCB KiCad project (motor-only board), linked to Kicad_Libs
- Controller: schematic, PCB and project updates
Parts:
- added C12: 1u, eCapacitor:0603, symbol Device:C
Connections:
- net C1: now also J6.4 (Pin_4); no longer J6.1 (Pin_1)
- net C2: now also J6.3 (Pin_3); no longer J6.2 (Pin_2)
- net C3: now also J6.1 (Pin_1); no longer J6.4 (Pin_4)
- net C4: now also J6.2 (Pin_2); no longer J6.3 (Pin_3)
- net D1: now also J6.8 (Pin_8); no longer J6.5 (Pin_5)
- net D2: now also J6.7 (Pin_7); no longer J6.6 (Pin_6)
- net D3: now also J6.5 (Pin_5); no longer J6.8 (Pin_8)
- net D4: now also J6.6 (Pin_6); no longer J6.7 (Pin_7)
- net G1: now also J7.4 (Pin_4); no longer J7.1 (Pin_1)
- net G2: now also J7.3 (Pin_3); no longer J7.2 (Pin_2)
- net G3: now also J7.1 (Pin_1); no longer J7.4 (Pin_4)
- net G4: now also J7.2 (Pin_2); no longer J7.3 (Pin_3)
- net GND: now also C12.2
- net H1: now also J7.8 (Pin_8); no longer J7.5 (Pin_5)
- net H2: now also J7.7 (Pin_7); no longer J7.6 (Pin_6)
- net H3: now also J7.5 (Pin_5); no longer J7.8 (Pin_8)
- net H4: now also J7.6 (Pin_6); no longer J7.7 (Pin_7)
- net at R5.2, SW2.1, U2.27 (IO0): now also C12.1
Other:
- moved on the sheet: SW2
Changed lines of the file:
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@@
 	)
 	(junction
+		(at 231.14 72.39)
+		(diameter 0)
+		(color 0 0 0 0)
+	)
+	(junction
 		(at 106.68 62.23)
 		(diameter 0)
@@
 	)
 	(junction
-		(at 231.14 72.39)
+		(at 321.31 166.37)
 		(diameter 0)
 		(color 0 0 0 0)
 	)
 	(junction
-		(at 321.31 166.37)
+		(at 130.81 233.68)
 		(diameter 0)
 		(color 0 0 0 0)
 	)
 	(junction
-		(at 130.81 233.68)
+		(at 85.09 62.23)
 		(diameter 0)
 		(color 0 0 0 0)
 	)
 	(junction
-		(at 85.09 62.23)
+		(at 226.06 72.39)
 		(diameter 0)
 		(color 0 0 0 0)
@@
 	(wire
 		(pts
-			(xy 201.93 72.39) (xy 231.14 72.39)
+			(xy 201.93 72.39) (xy 226.06 72.39)
 		)
 		(stroke
@@
 	(wire
 		(pts
+			(xy 226.06 92.71) (xy 226.06 91.44)
+		)
+		(stroke
+			(width 0)
+			(type default)
+		)
+	)
+	(wire
+		(pts
 			(xy 82.55 203.2) (xy 86.36 203.2)
 		)
@@
 	(wire
 		(pts
+			(xy 226.06 83.82) (xy 226.06 72.39)
+		)
+		(stroke
+			(width 0)
+			(type default)
+		)
+	)
+	(wire
+		(pts
 			(xy 331.47 227.33) (xy 336.55 227.33)
 		)
@@
 	(wire
 		(pts
+			(xy 234.95 72.39) (xy 231.14 72.39)
+		)
+		(stroke
+			(width 0)
+			(type default)
+		)
+	)
+	(wire
+		(pts
 			(xy 133.35 113.03) (xy 171.45 113.03)
 		)
@@
 	(wire
 		(pts
-			(xy 231.14 85.09) (xy 231.14 87.63)
+			(xy 234.95 91.44) (xy 234.95 93.98)
 		)
 		(stroke
@@
 	(wire
 		(pts
-			(xy 231.14 72.39) (xy 231.14 74.93)
+			(xy 234.95 72.39) (xy 234.95 81.28)
 		)
 		(stroke
@@
 	(wire
 		(pts
+			(xy 226.06 72.39) (xy 231.14 72.39)
+		)
+		(stroke
+			(width 0)
+			(type default)
+		)
+	)
+	(wire
+		(pts
 			(xy 295.91 229.87) (xy 298.45 229.87)
 		)
@@
 		)
 	)
-	(label "D2"
+	(label "D4"
 		(at 372.11 205.74 180)
 		(effects
@@
 		)
 	)
-	(label "H2"
+	(label "H4"
 		(at 372.11 229.87 180)
 		(effects
@@
 		)
 	)
-	(label "D4"
+	(label "D2"
 		(at 372.11 208.28 180)
 		(effects
@@
 		)
 	)
-	(label "D1"
+	(label "D3"
 		(at 372.11 203.2 180)
 		(effects
@@
 		)
 	)
-	(label "G4"
+	(label "G2"
 		(at 372.11 222.25 180)
 		(effects
@@
 		)
 	)
-	(label "C3"
+	(label "C1"
 		(at 372.11 200.66 180)
 		(effects
@@
 		)
 	)
-	(label "C1"
+	(label "C3"
 		(at 372.11 193.04 180)
 		(effects
@@
 		)
 	)
-	(label "H3"
+	(label "H1"
 		(at 372.11 234.95 180)
 		(effects
@@
 		)
 	)
-	(label "H4"
+	(label "H2"
 		(at 372.11 232.41 180)
 		(effects
@@
 		)
 	)
-	(label "C2"
+	(label "C4"
 		(at 372.11 195.58 180)
 		(effects
@@
 		)
 	)
-	(label "D3"
+	(label "D1"
 		(at 372.11 210.82 180)
 		(effects
@@
 		)
 	)
-	(label "H1"
+	(label "H3"
 		(at 372.11 227.33 180)
 		(effects
@@
 		)
 	)
-	(label "G2"
+	(label "G4"
 		(at 372.11 219.71 180)
 		(effects
@@
 		)
 	)
-	(label "G3"
+	(label "G1"
 		(at 372.11 224.79 180)
 		(effects
@@
 		)
 	)
-	(label "C4"
+	(label "C2"
 		(at 372.11 198.12 180)
 		(effects
@@
 		)
 	)
-	(label "G1"
+	(label "G3"
 		(at 372.11 217.17 180)
 		(effects
@@
 	(symbol
 		(lib_id "power:GND")
-		(at 231.14 87.63 0)
+		(at 234.95 93.98 0)
 		(mirror y)
 		(unit 1)
@@
 		(fields_autoplaced yes)
 		(property "Reference" "#PWR018"
-			(at 231.14 93.98 0)
+			(at 234.95 100.33 0)
 			(hide yes)
 			(show_name no)
@@
 		)
 		(property "Value" "GND"
-			(at 231.14 92.71 0)
+			(at 234.95 99.06 0)
 			(show_name no)
 			(do_not_autoplace no)
@@
 		)
 		(property "Footprint" ""
-			(at 231.14 87.63 0)
+			(at 234.95 93.98 0)
 			(hide yes)
 			(show_name no)
@@
 		)
 		(property "Datasheet" ""
-			(at 231.14 87.63 0)
+			(at 234.95 93.98 0)
 			(hide yes)
 			(show_name no)
@@
 		)
 		(property "Description" "Power symbol creates a global label with name \"GND\" , ground"
-			(at 231.14 87.63 0)
+			(at 234.95 93.98 0)
 			(hide yes)
 			(show_name no)
@@
 	)
 	(symbol
+		(lib_id "Device:C")
+		(at 226.06 87.63 0)
+		(mirror y)
+		(unit 1)
+		(body_style 1)
+		(exclude_from_sim no)
+		(in_bom yes)
+		(on_board yes)
+		(in_pos_files yes)
+		(dnp no)
+		(property "Reference" "C12"
+			(at 229.108 86.868 0)
+			(show_name no)
+			(do_not_autoplace no)
+			(effects
+				(font
+					(size 1.27 1.27)
+				)
+				(justify right)
+			)
+		)
+		(property "Value" "1u"
+			(at 229.87 88.8999 0)
+			(show_name no)
+			(do_not_autoplace no)
+			(effects
+				(font
+					(size 1.27 1.27)
+				)
+				(justify right)
+			)
+		)
+		(property "Footprint" "eCapacitor:0603"
+			(at 225.0948 91.44 0)
+			(hide yes)
+			(show_name no)
+			(do_not_autoplace no)
+			(effects
+				(font
+					(size 1.27 1.27)
+				)
+			)
+		)
+		(property "Datasheet" ""
+			(at 226.06 87.63 0)
+			(hide yes)
+			(show_name no)
+			(do_not_autoplace no)
+			(effects
+				(font
+					(size 1.27 1.27)
+				)
+			)
+		)
+		(property "Description" "Unpolarized capacitor"
+			(at 226.06 87.63 0)
+			(hide yes)
+			(show_name no)
+			(do_not_autoplace no)
+			(effects
+				(font
+					(size 1.27 1.27)
+				)
+			)
+		)
+		(pin "2"
+		)
+		(pin "1"
+		)
+		(instances
+			(project "ClockClock24"
+				(path "/6da799c4-65fe-48f3-b2d5-a73019f782b0"
+					(reference "C12")
+					(unit 1)
+				)
+			)
+		)
+	)
+	(symbol
 		(lib_id "power:GND")
 		(at 222.25 246.38 0)
@@
 	)
 	(symbol
+		(lib_id "power:GND")
+		(at 226.06 92.71 0)
+		(mirror y)
+		(unit 1)
+		(body_style 1)
+		(exclude_from_sim no)
+		(in_bom yes)
+		(on_board yes)
+		(in_pos_files yes)
+		(dnp no)
+		(fields_autoplaced yes)
+		(property "Reference" "#PWR036"
+			(at 226.06 99.06 0)
+			(hide yes)
+			(show_name no)
+			(do_not_autoplace no)
+			(effects
+				(font
+					(size 1.27 1.27)
+				)
+			)
+		)
+		(property "Value" "GND"
+			(at 226.06 97.79 0)
+			(show_name no)
+			(do_not_autoplace no)
+			(effects
+				(font
+					(size 1.27 1.27)
+				)
+			)
+		)
+		(property "Footprint" ""
+			(at 226.06 92.71 0)
+			(hide yes)
+			(show_name no)
+			(do_not_autoplace no)
+			(effects
+				(font
+					(size 1.27 1.27)
+				)
+			)
+		)
+		(property "Datasheet" ""
+			(at 226.06 92.71 0)
+			(hide yes)
+			(show_name no)
+			(do_not_autoplace no)
+			(effects
+				(font
+					(size 1.27 1.27)
+				)
+			)
+		)
+		(property "Description" "Power symbol creates a global label with name \"GND\" , ground"
+			(at 226.06 92.71 0)
+			(hide yes)
+			(show_name no)
+			(do_not_autoplace no)
+			(effects
+				(font
+					(size 1.27 1.27)
+				)
+			)
+		)
+		(pin "1"
+		)
+		(instances
+			(project "ClockClock24"
+				(path "/6da799c4-65fe-48f3-b2d5-a73019f782b0"
+					(reference "#PWR036")
+					(unit 1)
+				)
+			)
+		)
+	)
+	(symbol
 		(lib_id "Connector_Generic:Conn_01x08")
 		(at 303.53 200.66 0)
@@
 	(symbol
 		(lib_id "Switch:SW_Push")
-		(at 231.14 80.01 270)
+		(at 234.95 86.36 270)
 		(unit 1)
 		(body_style 1)
@@
 		(fields_autoplaced yes)
 		(property "Reference" "SW2"
-			(at 238.76 80.01 0)
+			(at 242.57 86.36 0)
 			(show_name no)
 			(do_not_autoplace no)
@@
 		)
 		(property "Value" "SW_Push"
-			(at 236.22 80.01 0)
+			(at 240.03 86.36 0)
 			(show_name no)
 			(do_not_autoplace no)
@@
 		)
 		(property "Footprint" "Button_Switch_SMD:SW_SPST_B3U-1000P"
-			(at 236.22 80.01 0)
+			(at 240.03 86.36 0)
 			(hide yes)
 			(show_name no)
@@
 		)
 		(property "Datasheet" ""
-			(at 236.22 80.01 0)
+			(at 240.03 86.36 0)
 			(hide yes)
 			(show_name no)
@@
 		)
 		(property "Description" "Push button switch, generic, two pins"
-			(at 231.14 80.01 0)
+			(at 234.95 86.36 0)
 			(hide yes)
 			(show_name no)

Commit message: Added Fab files, BOM and minor changes in layout
Parts:
- C1: LCSC (none) -> C19702
- C10, C2, C7, C8, C9: LCSC (none) -> C66501
- C11, C6: LCSC (none) -> C7469933
- C12, C3: LCSC (none) -> C1592
- C4, C5: LCSC (none) -> C19666
- D2: LCSC (none) -> C113952
- D3: LCSC (none) -> C22371297
- F1: LCSC (none) -> C269119
- J1: LCSC (none) -> C165948
- J2, J3: LCSC (none) -> C157972
- J4, J5, J6, J7: LCSC (none) -> C157974
- R1, R2: LCSC (none) -> C23186
- R10: LCSC (none) -> C105881
- R11: LCSC (none) -> C22548
- R12, R13: LCSC (none) -> C99782
- R14, R3, R4, R5: LCSC (none) -> C98220
- R9: LCSC (none) -> C14675
- SW1, SW2: LCSC (none) -> C231329
- U1: LCSC (none) -> C7519
- U2: LCSC (none) -> C2913198
- U3: LCSC (none) -> C500795
